File: schematic/motocamera_V1/motocamera_V1.kicad_sch (KiCad schematic)
At the start: 17 parts, among them J1 Raspberry_Pi_zero2W, SW1 SW_DIP_x06, SW2 SW_shutdown, U1 LM397, U3 LBR-123F

Commit message: 回路図修正
Parts:
- removed U3: LBR-123F, Crockwork_Cinecamera:LBR-123F, symbol crockwork_cinecamera:LBR-123F
- added U3: LBR-123F, OptoDevice:Letex_Technology_LBR-123F, symbol lbr-123f:LBR-123F
Connections:
- net +5V: now also U3.4
- net GND: now also U3.2 (K)
- net at R4.1, R5.1: now also U3.3
- net at R7.2: now also U3.1 (A)
Changed lines of the file:
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@@
     (stroke (width 0) (type default))
   )
-  (wire (pts (xy 260.35 45.72) (xy 260.35 92.71))
+  (wire (pts (xy 260.35 46.99) (xy 260.35 92.71))
     (stroke (width 0) (type default))
   )
@@
     (stroke (width 0) (type default))
   )
-  (wire (pts (xy 92.71 52.07) (xy 132.08 52.07))
-    (stroke (width 0) (type default))
-  )
   (wire (pts (xy 190.5 142.24) (xy 257.81 142.24))
     (stroke (width 0) (type default))
@@
     (stroke (width 0) (type default))
   )
-  (wire (pts (xy 92.71 45.72) (xy 260.35 45.72))
+  (wire (pts (xy 132.08 46.99) (xy 260.35 46.99))
     (stroke (width 0) (type default))
   )
@@
     (stroke (width 0) (type default))
   )
-  (wire (pts (xy 132.08 52.07) (xy 132.08 57.15))
+  (wire (pts (xy 132.08 46.99) (xy 132.08 57.15))
     (stroke (width 0) (type default))
   )
@@
   )
   (wire (pts (xy 200.66 134.62) (xy 200.66 85.09))
-    (stroke (width 0) (type default))
-  )
-  (wire (pts (xy 92.71 45.72) (xy 92.71 52.07))
     (stroke (width 0) (type default))
   )
@@
     )
   )
+  (symbol (lib_id "lbr-123f:LBR-123F") (at 53.34 88.9 0) (unit 1)
+    (in_bom yes) (on_board yes) (dnp no) (fields_autoplaced)
+    (property "Reference" "U3" (at 53.34 80.01 0)
+      (effects (font (size 1.27 1.27)))
+    )
+    (property "Value" "LBR-123F" (at 53.34 82.55 0)
+      (effects (font (size 1.27 1.27)))
+    )
+    (property "Footprint" "OptoDevice:Letex_Technology_LBR-123F" (at 53.34 96.52 0)
+      (effects (font (size 1.27 1.27)) hide)
+    )
+    (property "Datasheet" "https://akizukidenshi.com/goodsaffix/lbr-123f.pdf" (at 54.61 80.01 0)
+      (effects (font (size 1.27 1.27)) hide)
+    )
+    (pin "1")
+    (pin "4")
+    (pin "3")
+    (pin "2")
+    (instances
+      (project "motocamera_V1"
+        (path "/f6d74865-d282-4d13-b183-4c6ee03fe066"
+          (reference "U3") (unit 1)
+        )
+      )
+    )
+  )
   (symbol (lib_id "power:+5V") (at 93.98 44.45 0) (unit 1)
     (in_bom yes) (on_board yes) (dnp no) (fields_autoplaced)
@@
         )
       )
-    )
-  )
-  (symbol (lib_id "crockwork_cinecamera:LBR-123F") (at 53.34 88.9 0) (unit 1)
-    (in_bom yes) (on_board yes) (dnp no) (fields_autoplaced)
-    (property "Reference" "U3" (at 53.34 80.01 0)
-      (effects (font (size 1.27 1.27)))
-    )
-    (property "Value" "LBR-123F" (at 53.34 82.55 0)
-      (effects (font (size 1.27 1.27)))
-    )
-    (property "Footprint" "Crockwork_Cinecamera:LBR-123F" (at 53.34 96.52 0)
-      (effects (font (size 1.27 1.27)) hide)
-    )
-    (property "Datasheet" "https://akizukidenshi.com/goodsaffix/lbr-123f.pdf" (at 54.61 80.01 0)
-      (effects (font (size 1.27 1.27)) hide)
-    )
-    (pin "4")
-    (pin "3")
-    (pin "2")
-    (pin "1")
-    (instances
-      (project "motocamera_V1"
-        (path "/f6d74865-d282-4d13-b183-4c6ee03fe066"
-          (reference "U3") (unit 1)
-        )
-      )
