File: schematic/yashica8/yashica8.kicad_pcb (KiCad board)
At the start: 2 copper layers, 56.1 x 53.6 mm, 21 parts, among them J1 Raspberry_Pi_zero2W, SW1 SW_DIP_x06, SW2 SW_shutdown, U1 LM397, U3 LBR-123F_2

Commit message: cinemax8基板設計
Routing:
- net +5V: track 113.1 -> 128.5 mm, vias 2 -> 4
- net GND: vias 83 -> 75
Changed lines of the file:
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@@
   (via (at 124.46 99.06) (size 0.605) (drill 0.3) (layers "F.Cu" "B.Cu") (free) (net 1))
   (via (at 139.7 92.71) (size 0.605) (drill 0.3) (layers "F.Cu" "B.Cu") (free) (net 1))
-  (via (at 135.89 97.79) (size 0.605) (drill 0.3) (layers "F.Cu" "B.Cu") (free) (net 1))
   (via (at 116.84 88.9) (size 0.605) (drill 0.3) (layers "F.Cu" "B.Cu") (free) (net 1))
   (via (at 116.84 83.82) (size 0.605) (drill 0.3) (layers "F.Cu" "B.Cu") (free) (net 1))
   (via (at 149.86 85.09) (size 0.605) (drill 0.3) (layers "F.Cu" "B.Cu") (free) (net 1))
   (via (at 104.14 86.36) (size 0.605) (drill 0.3) (layers "F.Cu" "B.Cu") (free) (net 1))
-  (via (at 151.13 97.79) (size 0.605) (drill 0.3) (layers "F.Cu" "B.Cu") (free) (net 1))
   (via (at 116.84 96.52) (size 0.605) (drill 0.3) (layers "F.Cu" "B.Cu") (free) (net 1))
   (via (at 144.78 76.2) (size 0.605) (drill 0.3) (layers "F.Cu" "B.Cu") (free) (net 1))
@@
   (via (at 139.7 90.17) (size 0.605) (drill 0.3) (layers "F.Cu" "B.Cu") (free) (net 1))
   (via (at 106.68 111.76) (size 0.605) (drill 0.3) (layers "F.Cu" "B.Cu") (free) (net 1))
-  (via (at 143.51 97.79) (size 0.605) (drill 0.3) (layers "F.Cu" "B.Cu") (free) (net 1))
   (via (at 119.38 86.36) (size 0.605) (drill 0.3) (layers "F.Cu" "B.Cu") (free) (net 1))
   (via (at 114.3 76.2) (size 0.605) (drill 0.3) (layers "F.Cu" "B.Cu") (free) (net 1))
@@
   (via (at 139.7 87.63) (size 0.605) (drill 0.3) (layers "F.Cu" "B.Cu") (free) (net 1))
   (via (at 105.41 115.57) (size 0.605) (drill 0.3) (layers "F.Cu" "B.Cu") (free) (net 1))
-  (via (at 124.46 93.98) (size 0.605) (drill 0.3) (layers "F.Cu" "B.Cu") (free) (net 1))
   (via (at 143.51 92.71) (size 0.605) (drill 0.3) (layers "F.Cu" "B.Cu") (free) (net 1))
   (via (at 151.13 95.25) (size 0.605) (drill 0.3) (layers "F.Cu" "B.Cu") (free) (net 1))
-  (via (at 124.46 88.9) (size 0.605) (drill 0.3) (layers "F.Cu" "B.Cu") (free) (net 1))
   (via (at 129.54 93.98) (size 0.605) (drill 0.3) (layers "F.Cu" "B.Cu") (free) (net 1))
   (via (at 127 91.44) (size 0.605) (drill 0.3) (layers "F.Cu" "B.Cu") (free) (net 1))
   (via (at 147.32 87.63) (size 0.605) (drill 0.3) (layers "F.Cu" "B.Cu") (free) (net 1))
   (via (at 129.54 81.28) (size 0.605) (drill 0.3) (layers "F.Cu" "B.Cu") (free) (net 1))
-  (via (at 129.54 99.06) (size 0.605) (drill 0.3) (layers "F.Cu" "B.Cu") (free) (net 1))
-  (via (at 139.7 97.79) (size 0.605) (drill 0.3) (layers "F.Cu" "B.Cu") (free) (net 1))
   (via (at 106.68 88.9) (size 0.605) (drill 0.3) (layers "F.Cu" "B.Cu") (free) (net 1))
   (via (at 111.76 78.74) (size 0.605) (drill 0.3) (layers "F.Cu" "B.Cu") (free) (net 1))
@@
   (via (at 105.41 120.65) (size 0.605) (drill 0.3) (layers "F.Cu" "B.Cu") (free) (net 1))
   (via (at 106.68 78.74) (size 0.605) (drill 0.3) (layers "F.Cu" "B.Cu") (free) (net 1))
-  (via (at 147.32 97.79) (size 0.605) (drill 0.3) (layers "F.Cu" "B.Cu") (free) (net 1))
   (via (at 137.16 101.6) (size 0.605) (drill 0.3) (layers "F.Cu" "B.Cu") (free) (net 1))
   (via (at 143.51 95.25) (size 0.605) (drill 0.3) (layers "F.Cu" "B.Cu") (free) (net 1))
@@
   (segment (start 147.05 106.41) (end 148.59 106.41) (width 0.2) (layer "F.Cu") (net 3))
   (segment (start 146.05 105.41) (end 147.05 106.41) (width 0.2) (layer "F.Cu") (net 3))
+  (segment (start 120.65 90.17) (end 123.19 90.17) (width 0.6) (layer "F.Cu") (net 5))
   (segment (start 103.9924 108.8024) (end 103.14 107.95) (width 0.2) (layer "F.Cu") (net 5))
   (segment (start 103.14 105.41) (end 103.14 107.95) (width 0.2) (layer "F.Cu") (net 5))
   (segment (start 117.5576 90.2576) (end 118.11 90.81) (width 0.2) (layer "F.Cu") (net 5))
   (segment (start 106.95 91.44) (end 108.1324 90.2576) (width 0.2) (layer "F.Cu") (net 5))
-  (segment (start 120.01 90.81) (end 123.19 87.63) (width 0.6) (layer "F.Cu") (net 5))
-  (segment (start 123.19 86.36) (end 123.19 87.63) (width 0.6) (layer "F.Cu") (net 5))
+  (segment (start 151.13 118.11) (end 152.4 119.38) (width 2) (layer "F.Cu") (net 5))
+  (segment (start 123.19 91.44) (end 123.19 93.98) (width 2) (layer "F.Cu") (net 5))
   (segment (start 107.95 124.46) (end 103.9924 120.5024) (width 0.2) (layer "F.Cu") (net 5))
-  (segment (start 120.01 90.81) (end 123.83 90.81) (width 0.6) (layer "F.Cu") (net 5))
-  (segment (start 153.67 119.38) (end 151.13 116.84) (width 0.6) (layer "F.Cu") (net 5))
-  (segment (start 153.67 121.92) (end 153.67 119.38) (width 0.6) (layer "F.Cu") (net 5))
+  (segment (start 152.4 120.65) (end 153.67 121.92) (width 2) (layer "F.Cu") (net 5))
+  (segment (start 123.19 87.63) (end 123.19 90.17) (width 2) (layer "F.Cu") (net 5))
+  (segment (start 152.4 119.38) (end 153.67 119.38) (width 2) (layer "F.Cu") (net 5))
   (segment (start 118.11 90.81) (end 120.01 90.81) (width 0.6) (layer "F.Cu") (net 5))
   (segment (start 103.14 105.41) (end 103.14 95.25) (width 0.2) (layer "F.Cu") (net 5))
   (segment (start 108.1324 90.2576) (end 117.5576 90.2576) (width 0.2) (layer "F.Cu") (net 5))
   (segment (start 103.14 95.25) (end 106.95 91.44) (width 0.2) (layer "F.Cu") (net 5))
-  (segment (start 123.83 90.81) (end 125.73 92.71) (width 0.6) (layer "F.Cu") (net 5))
+  (segment (start 123.19 90.17) (end 123.19 91.44) (width 2) (layer "F.Cu") (net 5))
+  (segment (start 120.01 90.81) (end 120.65 90.17) (width 0.6) (layer "F.Cu") (net 5))
+  (segment (start 123.19 86.36) (end 123.19 87.63) (width 2) (layer "F.Cu") (net 5))
+  (segment (start 151.13 120.65) (end 152.4 120.65) (width 2) (layer "F.Cu") (net 5))
   (segment (start 103.9924 120.5024) (end 103.9924 108.8024) (width 0.2) (layer "F.Cu") (net 5))
-  (via (at 151.13 116.84) (size 0.605) (drill 0.3) (layers "F.Cu" "B.Cu") (net 5))
-  (via (at 125.73 92.71) (size 0.605) (drill 0.3) (layers "F.Cu" "B.Cu") (net 5))
-  (segment (start 151.13 101.6) (end 148.59 99.06) (width 0.6) (layer "B.Cu") (net 5))
-  (segment (start 148.59 99.06) (end 147.32 99.06) (width 0.6) (layer "B.Cu") (net 5))
-  (segment (start 132.08 99.06) (end 125.73 92.71) (width 0.6) (layer "B.Cu") (net 5))
-  (segment (start 137.16 99.06) (end 132.08 99.06) (width 0.6) (layer "B.Cu") (net 5))
-  (segment (start 151.13 101.6) (end 151.13 116.84) (width 0.6) (layer "B.Cu") (net 5))
-  (segment (start 142.24 99.06) (end 137.16 99.06) (width 0.6) (layer "B.Cu") (net 5))
-  (segment (start 147.32 99.06) (end 142.24 99.06) (width 0.6) (layer "B.Cu") (net 5))
+  (via (at 123.19 93.98) (size 1.5) (drill 1) (layers "F.Cu" "B.Cu") (net 5))
+  (via (at 151.13 120.65) (size 1.5) (drill 1) (layers "F.Cu" "B.Cu") (net 5))
+  (via (at 151.13 118.11) (size 1.5) (drill 1) (layers "F.Cu" "B.Cu") (net 5))
+  (via (at 123.19 91.44) (size 1.5) (drill 1) (layers "F.Cu" "B.Cu") (net 5))
+  (segment (start 148.59 99.06) (end 151.13 101.6) (width 2) (layer "B.Cu") (net 5))
+  (segment (start 151.13 101.6) (end 151.13 118.11) (width 2) (layer "B.Cu") (net 5))
+  (segment (start 123.19 91.44) (end 130.81 99.06) (width 2) (layer "B.Cu") (net 5))
+  (segment (start 130.81 99.06) (end 148.59 99.06) (width 2) (layer "B.Cu") (net 5))
+  (segment (start 151.13 118.11) (end 151.13 120.65) (width 2) (layer "B.Cu") (net 5))
+  (segment (start 123.19 93.98) (end 128.27 99.06) (width 2) (layer "B.Cu") (net 5))
+  (segment (start 128.27 99.06) (end 130.81 99.06) (width 2) (layer "B.Cu") (net 5))
   (segment (start 108.95 93.98) (end 116.84 93.98) (width 0.2) (layer "F.Cu") (net 15))
   (segment (start 108.95 93.98) (end 108.95 91.44) (width 0.2) (layer "F.Cu") (net 15))
