File: schematic/cinemax8/cinemax8.kicad_pcb (KiCad board)
At the start: 2 copper layers, 58.9 x 48.8 mm, 21 parts, among them J1 Raspberry_Pi_zero2W, SW1 SW_DIP_x06, SW2 SW_shutdown, U1 LM397, U3 LBR-123F_2

Commit message: 基板設計
Parts:
- moved R2 1.27 mm to (132.1, 85.1)
- moved R3 1.27 mm to (132.1, 82.5)
- moved R6 1.27 mm to (132.1, 80.0)
Connections:
- U3 pad 3: +5V -> Net-(R4-Pad1)
- U3 pad 4: Net-(R4-Pad1) -> +5V
Routing:
- net Net-(R4-Pad1): track 17.1 -> 14.5 mm
- net +5V: track 134.9 -> 137.2 mm
- net Net-(J1-GPIO25): track 72.6 -> 74.5 mm
- net Net-(U1-+): track 30.7 -> 31.9 mm
- net GND: vias 82 -> 75
Other:
- outline, holes or cut-outs redrawn
