File: schematic/yashica8_ver0.1.1/yashica8_ver0.1.1.kicad_pcb (KiCad board)
At the start: 2 copper layers, 56.1 x 53.6 mm, 24 parts, among them J1 Raspberry_Pi_zero2W, J2 9V, J3 GND, SW1 SW_DIP_x06, SW2 SW_shutdown, SW3 SS-012D0, U1 LM397, U3 LBR-123F_2

Commit message: board 0.1.2 added
Parts:
- J2: value 9V -> 9V Pad
- J3: value GND -> GND Pad
- U2: footprint Crockwork_Cinecamera:MP2307 DC-DC Board -> clock_work_camera:MP2307 DC-DC Board
- moved D1 1.27 mm to (144.8, 111.8)
- moved D2 1.27 mm to (144.8, 106.7)
- moved R8 1.27 mm to (149.9, 111.4)
- moved R9 1.27 mm to (149.9, 106.3)
- moved U2 0.64 mm to (108.0, 85.7)
Routing:
- net Net-(J1-GPIO15/RXD): track 5.66 -> 4.39 mm
- net Net-(J1-GPIO18/PWM0): track 6.71 -> 5.52 mm
- net +5V: track 133.4 -> 134.2 mm
- net Net-(U2-IN+): track 3.81 -> 4.47 mm
