File: schematic/yashica8_ver0.1.2/yashica8_ver0.1.2.kicad_sch (KiCad schematic)
At the start: 24 parts, among them J1 Raspberry_Pi_zero2W, J2 9V Pad, J3 GND Pad, SW1 SW_DIP_x06, SW2 SW_shutdown, SW3 SS-012D0, U1 LM397, U3 LBR-123F_2

Commit message: board 0.1.2 added
Parts:
- removed SW3: SS-012D0, clock_work_camera:slide_switch, symbol crockwork_cinecamera:slide_switch
- added SW3: IS-2235-G, clock_work_camera:IS-2235-G, symbol crockwork_cinecamera:IS-2235-G
Connections:
- net +9V: now also SW3.2 (B), SW3.5 (B)
- net at U2.1 (IN+): now also SW3.1 (A), SW3.4 (C)
- no-connect marks 20 -> 22
Changed lines of the file:
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@@
+	)
+	(junction
+		(at 110.49 152.4)
+		(diameter 0)
+		(color 0 0 0 0)
 	)
 	(junction
@@
 		(color 0 0 0 0)
 	)
+	(junction
+		(at 92.71 142.24)
+		(diameter 0)
+		(color 0 0 0 0)
+	)
 	(no_connect
 		(at 247.65 64.77)
 	)
 	(no_connect
+		(at 93.98 157.48)
+	)
+	(no_connect
 		(at 247.65 107.95)
-	)
-	(no_connect
-		(at 92.71 147.32)
 	)
 	(no_connect
@@
 	)
 	(no_connect
+		(at 116.84 158.75)
+	)
+	(no_connect
 		(at 247.65 97.79)
 	)
@@
 	)
 	(no_connect
+		(at 104.14 157.48)
+	)
+	(no_connect
 		(at 247.65 82.55)
 	)
@@
 	(wire
 		(pts
+			(xy 91.44 160.02) (xy 110.49 160.02)
+		)
+		(stroke
+			(width 0)
+			(type default)
+		)
+	)
+	(wire
+		(pts
 			(xy 227.33 120.65) (xy 227.33 123.19)
 		)
@@
 	(wire
 		(pts
+			(xy 104.14 142.24) (xy 104.14 147.32)
+		)
+		(stroke
+			(width 0)
+			(type default)
+		)
+	)
+	(wire
+		(pts
 			(xy 234.95 123.19) (xy 234.95 120.65)
 		)
@@
 	(wire
 		(pts
+			(xy 93.98 152.4) (xy 91.44 152.4)
+		)
+		(stroke
+			(width 0)
+			(type default)
+		)
+	)
+	(wire
+		(pts
 			(xy 217.17 123.19) (xy 217.17 125.73)
 		)
@@
 	(wire
 		(pts
+			(xy 91.44 152.4) (xy 91.44 160.02)
+		)
+		(stroke
+			(width 0)
+			(type default)
+		)
+	)
+	(wire
+		(pts
 			(xy 93.98 44.45) (xy 93.98 50.8)
 		)
@@
 	(wire
 		(pts
+			(xy 92.71 142.24) (xy 104.14 142.24)
+		)
+		(stroke
+			(width 0)
+			(type default)
+		)
+	)
+	(wire
+		(pts
 			(xy 154.94 132.08) (xy 175.26 132.08)
 		)
@@
 	(wire
 		(pts
+			(xy 92.71 147.32) (xy 92.71 142.24)
+		)
+		(stroke
+			(width 0)
+			(type default)
+		)
+	)
+	(wire
+		(pts
 			(xy 255.27 90.17) (xy 255.27 142.24)
 		)
@@
 	(wire
 		(pts
+			(xy 92.71 142.24) (xy 88.9 142.24)
+		)
+		(stroke
+			(width 0)
+			(type default)
+		)
+	)
+	(wire
+		(pts
 			(xy 132.08 64.77) (xy 132.08 68.58)
 		)
@@
 	(wire
 		(pts
+			(xy 104.14 152.4) (xy 110.49 152.4)
+		)
+		(stroke
+			(width 0)
+			(type default)
+		)
+	)
+	(wire
+		(pts
 			(xy 171.45 100.33) (xy 171.45 95.25)
 		)
@@
 	(wire
 		(pts
+			(xy 110.49 152.4) (xy 110.49 139.7)
+		)
+		(stroke
+			(width 0)
+			(type default)
+		)
+	)
+	(wire
+		(pts
 			(xy 224.79 120.65) (xy 224.79 123.19)
 		)
@@
 	(wire
 		(pts
-			(xy 88.9 142.24) (xy 92.71 142.24)
+			(xy 92.71 147.32) (xy 93.98 147.32)
 		)
 		(stroke
@@
 	(wire
 		(pts
-			(xy 105.41 144.78) (xy 110.49 144.78)
-		)
-		(stroke
-			(width 0)
-			(type default)
-		)
-	)
-	(wire
-		(pts
 			(xy 132.08 46.99) (xy 200.66 46.99)
 		)
@@
 	(wire
 		(pts
-			(xy 110.49 144.78) (xy 110.49 139.7)
-		)
-		(stroke
-			(width 0)
-			(type default)
-		)
-	)
-	(wire
-		(pts
 			(xy 198.12 85.09) (xy 198.12 132.08)
 		)
@@
 		(pts
 			(xy 219.71 123.19) (xy 222.25 123.19)
+		)
+		(stroke
+			(width 0)
+			(type default)
+		)
+	)
+	(wire
+		(pts
+			(xy 110.49 160.02) (xy 110.49 152.4)
 		)
 		(stroke
@@
 	)
 	(symbol
-		(lib_id "crockwork_cinecamera:slide_switch")
-		(at 99.06 144.78 0)
-		(unit 1)
-		(exclude_from_sim no)
-		(in_bom yes)
-		(on_board yes)
-		(dnp no)
-		(fields_autoplaced yes)
-		(property "Reference" "SW3"
-			(at 99.06 135.89 0)
-			(effects
-				(font
-					(size 1.27 1.27)
-				)
-			)
-		)
-		(property "Value" "SS-012D0"
-			(at 99.06 138.43 0)
-			(effects
-				(font
-					(size 1.27 1.27)
-				)
-			)
-		)
-		(property "Footprint" "clock_work_camera:slide_switch"
-			(at 99.06 144.78 0)
-			(effects
-				(font
-					(size 1.27 1.27)
-				)
-				(hide yes)
-			)
-		)
-		(property "Datasheet" ""
-			(at 99.06 144.78 0)
-			(effects
-				(font
-					(size 1.27 1.27)
-				)
-				(hide yes)
-			)
-		)
-		(property "Description" ""
-			(at 99.06 144.78 0)
-			(effects
-				(font
-					(size 1.27 1.27)
-				)
-				(hide yes)
-			)
-		)
-		(pin "1"
-		)
-		(pin "3"
-		)
-		(pin "2"
-		)
-		(instances
-			(project "yashica8_ver0.1.1"
-				(path "/f6d74865-d282-4d13-b183-4c6ee03fe066"
-					(reference "SW3")
-					(unit 1)
-				)
-			)
-		)
-	)
-	(symbol
 		(lib_id "Device:R")
 		(at 69.85 97.79 90)
@@
 					(unit 1)
 				)
+			)
+		)
+	)
+	(symbol
+		(lib_id "crockwork_cinecamera:IS-2235-G")
+		(at 99.06 152.4 0)
+		(unit 1)
+		(exclude_from_sim no)
+		(in_bom yes)
+		(on_board yes)
+		(dnp no)
+		(property "Reference" "SW3"
+			(at 99.06 161.798 0)
+			(effects
+				(font
+					(size 1.27 1.27)
+				)
+			)
+		)
+		(property "Value" "IS-2235-G"
+			(at 99.06 164.084 0)
+			(effects
+				(font
+					(size 1.27 1.27)
+				)
+			)
+		)
+		(property "Footprint" "clock_work_camera:IS-2235-G"
+			(at 113.03 147.32 0)
+			(effects
+				(font
+					(size 1.27 1.27)
+				)
+				(hide yes)
+			)
+		)
+		(property "Datasheet" "~"
+			(at 99.06 152.4 0)
+			(effects
+				(font
+					(size 1.27 1.27)
+				)
+				(hide yes)
+			)
+		)
+		(property "Description" "Slide Switch, dual pole double throw"
+			(at 99.06 152.4 0)
+			(effects
+				(font
+					(size 1.27 1.27)
+				)
+				(hide yes)
+			)
+		)
+		(pin "5"
+		)
+		(pin "1"
+		)
+		(pin "5"
+		)
+		(pin "2"
+		)
+		(pin "3"
+		)
+		(pin "4"
+		)
+		(instances
+			(project ""
+				(path "/f6d74865-d282-4d13-b183-4c6ee03fe066"
+					(reference "SW3")
+					(unit 1)
+				)
